Commit message: add ultrasonic sensor

File: src/jackal_description/urdf/accessories_two.urdf.xacro (robot description, xacro)
@@ -26,5 +26,5 @@
     optional microstrain IMU's will be added to another frame, by default, "microstrain_link".
   -->
-  <xacro:if value="$(optenv JACKAL_IMU_MICROSTRAIN 0)">
+  <xacro:if value="$(optenv JACKAL_IMU_MICROSTRAIN 1)">
     <xacro:property name="frame"  value="$(optenv JACKAL_IMU_MICROSTRAIN_LINK microstrain_link)"/>
     <xacro:property name="parent" value="$(optenv JACKAL_IMU_MICROSTRAIN_PARENT base_link)"/>
@@ -52,5 +52,5 @@
     <xacro:property name="prefix" value="$(optenv JACKAL_LASER_PREFIX ${mount}_high)" />
     <xacro:property name="parent" value="$(optenv JACKAL_LASER_PARENT ${mount}_mount_high)" />
-    <xacro:property name="lidar_model" value="$(optenv JACKAL_LASER_MODEL utm30)" />
+    <xacro:property name="lidar_model" value="$(optenv JACKAL_LASER_MODEL lms1xx)" />
     <xacro:property name="mount_type" value="$(optenv JACKAL_LASER_MOUNT_TYPE upright)" />
     <!-- SICK LMS1xx -->

File: src/jackal_description/urdf/jackal.urdf.xacro (robot description, xacro)
@@ -218,4 +218,10 @@
     <origin xyz="${mount_spacing} 0 0" />
   </joint>
+  <link name="ultrasonic_sensor_link"></link>
+  <joint name="ultrasonic_sensor_joint" type="fixed">
+    <parent link="front_mount"/>
+    <child link="ultrasonic_sensor_link"/>
+    <origin xyz="0.12 0 -0.2" />
+  </joint>
   <!-- Bring in simulation data for Gazebo. -->
   <xacro:include filename="$(find jackal_description)/urdf/jackal.gazebo" />

File: src/jackal_description/urdf/jackal_two.urdf.xacro (robot description, xacro)
@@ -222,5 +222,5 @@
     <parent link="mid_mount" />
     <child link="front_mount_high" />
-    <origin xyz="${mount_spacing} 0 0.1" />
+    <origin xyz="${mount_spacing} 0 0" />
   </joint>
   <link name="front_mount_low"></link>
