Commit message: before adding cam

File: src/jackal_description/urdf/accessories.urdf.xacro (robot description, xacro)
@@ -26,5 +26,5 @@
     optional microstrain IMU's will be added to another frame, by default, "microstrain_link".
   -->
-  <xacro:if value="$(optenv JACKAL_IMU_MICROSTRAIN 1)">
+  <xacro:if value="$(optenv JACKAL_IMU_MICROSTRAIN 0)">
     <xacro:property name="frame"  value="$(optenv JACKAL_IMU_MICROSTRAIN_LINK microstrain_link)"/>
     <xacro:property name="parent" value="$(optenv JACKAL_IMU_MICROSTRAIN_PARENT base_link)"/>
@@ -52,5 +52,5 @@
     <xacro:property name="prefix" value="$(optenv JACKAL_LASER_PREFIX ${mount})" />
     <xacro:property name="parent" value="$(optenv JACKAL_LASER_PARENT ${mount}_mount)" />
-    <xacro:property name="lidar_model" value="$(optenv JACKAL_LASER_MODEL tim551)" />
+    <xacro:property name="lidar_model" value="$(optenv JACKAL_LASER_MODEL utm30)" />
     <xacro:property name="mount_type" value="$(optenv JACKAL_LASER_MOUNT_TYPE upright)" />
     <!-- SICK LMS1xx -->
@@ -115,5 +115,5 @@
     <xacro:property name="prefix" value="$(optenv JACKAL_LASER_SECONDARY_PREFIX ${mount})" />
     <xacro:property name="parent" value="$(optenv JACKAL_LASER_SECONDARY_PARENT ${mount}_mount)" />
-    <xacro:property name="lidar_model" value="$(optenv JACKAL_LASER_SECONDARY_MODEL lms1xx)" />
+    <xacro:property name="lidar_model" value="$(optenv JACKAL_LASER_SECONDARY_MODEL utm30)" />
     <!-- SICK LMS1xx -->
     <xacro:if value="${lidar_model == 'lms1xx'}">

File: src/velodyne_description/urdf/HDL-32E.urdf.xacro (robot description, xacro)
@@ -2,5 +2,5 @@
 <robot xmlns:xacro="http://www.ros.org/wiki/xacro" name="HDL-32E">
   <xacro:property name="M_PI" value="3.1415926535897931" />
-  <xacro:macro name="HDL-32E" params="*origin parent:=base_link name:=velodyne topic:=/velodyne_points organize_cloud:=false hz:=10 lasers:=32 samples:=2187 collision_range:=0.3 min_range:=0.9 max_range:=130.0 noise:=0.008 min_angle:=-${M_PI} max_angle:=${M_PI} gpu:=false">
+  <xacro:macro name="HDL-32E" params="*origin parent:=base_link name:=velodyne topic:=/velodyne_points organize_cloud:=false hz:=10 lasers:=32 samples:=2187 collision_range:=0.3 min_range:=0.9 max_range:=130.0 noise:=0.008 min_angle:=-${M_PI} max_angle:=${M_PI} gpu:=true">
     <joint name="${name}_base_mount_joint" type="fixed">
       <xacro:insert_block name="origin" />

File: src/velodyne_description/urdf/VLP-16.urdf.xacro (robot description, xacro)
@@ -2,5 +2,5 @@
 <robot xmlns:xacro="http://www.ros.org/wiki/xacro" name="VLP-16">
   <xacro:property name="M_PI" value="3.1415926535897931" />
-  <xacro:macro name="VLP-16" params="*origin parent:=base_link name:=velodyne topic:=/velodyne_points organize_cloud:=false hz:=10 lasers:=16 samples:=1875 collision_range:=0.3 min_range:=0.9 max_range:=130.0 noise:=0.008 min_angle:=-${M_PI} max_angle:=${M_PI} gpu:=false">
+  <xacro:macro name="VLP-16" params="*origin parent:=base_link name:=velodyne topic:=/velodyne_points organize_cloud:=false hz:=10 lasers:=16 samples:=300 collision_range:=0.2 min_range:=0.2 max_range:=10.0 noise:=0.002 min_angle:=-${M_PI} max_angle:=${M_PI} gpu:=true">
     <joint name="${name}_base_mount_joint" type="fixed">
       <xacro:insert_block name="origin" />
@@ -67,5 +67,5 @@
               <horizontal>
                 <samples>${samples}</samples>
-                <resolution>1</resolution>
+                <resolution>30</resolution>
                 <min_angle>${min_angle}</min_angle>
                 <max_angle>${max_angle}</max_angle>
@@ -73,5 +73,5 @@
               <vertical>
                 <samples>${lasers}</samples>
-                <resolution>1</resolution>
+                <resolution>30</resolution>
                 <min_angle>-${15.0*M_PI/180.0}</min_angle>
                 <max_angle> ${15.0*M_PI/180.0}</max_angle>
@@ -108,5 +108,5 @@
               <horizontal>
                 <samples>${samples}</samples>
-                <resolution>1</resolution>
+                <resolution>30</resolution>
                 <min_angle>${min_angle}</min_angle>
                 <max_angle>${max_angle}</max_angle>
@@ -114,5 +114,5 @@
               <vertical>
                 <samples>${lasers}</samples>
-                <resolution>1</resolution>
+                <resolution>30</resolution>
                 <min_angle>-${15.0*M_PI/180.0}</min_angle>
                 <max_angle> ${15.0*M_PI/180.0}</max_angle>

Commit message: add jackal other pack

File: src/jackal_description/urdf/accessories.urdf.xacro (robot description, xacro)
@@ -169,5 +169,5 @@
     - vlp32e           :: Velodyne HDL-32E
   -->
-  <xacro:if value="$(optenv JACKAL_LASER_3D 1)">
+  <xacro:if value="$(optenv JACKAL_LASER_3D 0)">
     <xacro:property name="mount" value="$(optenv JACKAL_LASER_3D_MOUNT mid)" />
     <xacro:property name="topic" value="$(optenv JACKAL_LASER_3D_TOPIC mid/points)" />

File: src/jackal_description/urdf/accessories/hokuyo_utm30.urdf.xacro (robot description, xacro)
@@ -1,7 +1,7 @@
 <?xml version="1.0"?>
 <robot xmlns:xacro="http://ros.org/wiki/xacro">
-  <xacro:macro name="hokuyo_utm30_mount" params="prefix topic parent_link min_angle:=-2.2689  max_angle:=2.2689 *origin">
+  <xacro:macro name="hokuyo_utm30_mount" params="prefix topic parent_link min_angle:=-3  max_angle:=3 *origin">
     <xacro:macro name="hokuyo_utm30" params="frame:=laser topic:=scan sample_size:=1440 update_rate:=50
-               min_angle:=-2.2689 max_angle:=2.2689 min_range:=0.1 max_range:=30.0 robot_namespace:=/">
+               min_angle:=-3 max_angle:=3 min_range:=0.1 max_range:=30.0 robot_namespace:=/">
       <xacro:property name="mass" value="0.370"/>
       <xacro:property name="base" value="0.06" />

Commit message: two scan merge

File: src/jackal_description/urdf/accessories.urdf.xacro (robot description, xacro)
@@ -48,8 +48,8 @@
   <xacro:if value="$(optenv JACKAL_LASER 1)">
     <xacro:property name="mount" value="$(optenv JACKAL_LASER_MOUNT front)" />
-    <xacro:property name="topic" value="$(optenv JACKAL_LASER_TOPIC front/scan)" />
+    <xacro:property name="topic" value="$(optenv JACKAL_LASER_TOPIC front/scan1)" />
     <xacro:property name="tower" value="$(optenv JACKAL_LASER_TOWER 1)" />
-    <xacro:property name="prefix" value="$(optenv JACKAL_LASER_PREFIX ${mount})" />
-    <xacro:property name="parent" value="$(optenv JACKAL_LASER_PARENT ${mount}_mount)" />
+    <xacro:property name="prefix" value="$(optenv JACKAL_LASER_PREFIX ${mount}_high)" />
+    <xacro:property name="parent" value="$(optenv JACKAL_LASER_PARENT ${mount}_mount_high)" />
     <xacro:property name="lidar_model" value="$(optenv JACKAL_LASER_MODEL utm30)" />
     <xacro:property name="mount_type" value="$(optenv JACKAL_LASER_MOUNT_TYPE upright)" />
@@ -109,10 +109,10 @@
   </xacro:if>
   <!-- Secondary 2D Lidar -->
-  <xacro:if value="$(optenv JACKAL_LASER_SECONDARY 0)">
-    <xacro:property name="mount" value="$(optenv JACKAL_LASER_SECONDARY_MOUNT rear)" />
-    <xacro:property name="topic" value="$(optenv JACKAL_LASER_SECONDARY_TOPIC rear/scan)" />
+  <xacro:if value="$(optenv JACKAL_LASER_SECONDARY 1)">
+    <xacro:property name="mount" value="$(optenv JACKAL_LASER_SECONDARY_MOUNT front)" />
+    <xacro:property name="topic" value="$(optenv JACKAL_LASER_SECONDARY_TOPIC front/scan2)" />
     <xacro:property name="tower" value="$(optenv JACKAL_LASER_SECONDARY_TOWER 1)" />
-    <xacro:property name="prefix" value="$(optenv JACKAL_LASER_SECONDARY_PREFIX ${mount})" />
-    <xacro:property name="parent" value="$(optenv JACKAL_LASER_SECONDARY_PARENT ${mount}_mount)" />
+    <xacro:property name="prefix" value="$(optenv JACKAL_LASER_SECONDARY_PREFIX ${mount}_low)" />
+    <xacro:property name="parent" value="$(optenv JACKAL_LASER_SECONDARY_PARENT ${mount}_mount_low)" />
     <xacro:property name="lidar_model" value="$(optenv JACKAL_LASER_SECONDARY_MODEL utm30)" />
     <!-- SICK LMS1xx -->
@@ -159,5 +159,5 @@
     <xacro:if value="${lidar_model == 'utm30'}">
       <xacro:hokuyo_utm30_mount topic="${topic}" prefix="${prefix}" parent_link="${parent}">
-        <origin xyz="$(optenv JACKAL_LASER_SECONDARY_OFFSET 0 0 0)" rpy="$(optenv JACKAL_LASER_SECONDARY_RPY 0 0 3.14159)" />
+        <origin xyz="$(optenv JACKAL_LASER_SECONDARY_OFFSET 0 0 0)" rpy="$(optenv JACKAL_LASER_SECONDARY_RPY 0 0 0)" />
       </xacro:hokuyo_utm30_mount>
     </xacro:if>

File: src/jackal_description/urdf/accessories/hokuyo_utm30.urdf.xacro (robot description, xacro)
@@ -1,7 +1,7 @@
 <?xml version="1.0"?>
 <robot xmlns:xacro="http://ros.org/wiki/xacro">
-  <xacro:macro name="hokuyo_utm30_mount" params="prefix topic parent_link min_angle:=-3  max_angle:=3 *origin">
+  <xacro:macro name="hokuyo_utm30_mount" params="prefix topic parent_link min_angle:=-2.356194  max_angle:=2.356194 *origin">
     <xacro:macro name="hokuyo_utm30" params="frame:=laser topic:=scan sample_size:=1440 update_rate:=50
-               min_angle:=-3 max_angle:=3 min_range:=0.1 max_range:=30.0 robot_namespace:=/">
+               min_angle:=-2.356194 max_angle:=2.356194 min_range:=0.1 max_range:=30.0 robot_namespace:=/">
       <xacro:property name="mass" value="0.370"/>
       <xacro:property name="base" value="0.06" />

File: src/jackal_description/urdf/jackal.urdf.xacro (robot description, xacro)
@@ -218,4 +218,16 @@
     <origin xyz="${mount_spacing} 0 0" />
   </joint>
+  <link name="front_mount_high"></link>
+  <joint name="front_mount_joint_high" type="fixed">
+    <parent link="mid_mount" />
+    <child link="front_mount_high" />
+    <origin xyz="${mount_spacing} 0 0.1" />
+  </joint>
+  <link name="front_mount_low"></link>
+  <joint name="front_mount_joint_low" type="fixed">
+    <parent link="mid_mount" />
+    <child link="front_mount_low" />
+    <origin xyz="${mount_spacing} 0 -0.3" />
+  </joint>
   <!-- Bring in simulation data for Gazebo. -->
   <xacro:include filename="$(find jackal_description)/urdf/jackal.gazebo" />

Commit message: amcl alpha modified

File: src/jackal_description/urdf/accessories.urdf.xacro (robot description, xacro)
@@ -262,5 +262,5 @@
   <xacro:if value="$(optenv JACKAL_FLEA3 1)">
     <xacro:property name="name" value="$(optenv JACKAL_FLEA3_NAME front)" />
-    <xacro:property name="tilt" value="$(optenv JACKAL_FLEA3_TILT 0.5236)" />
+    <xacro:property name="tilt" value="$(optenv JACKAL_FLEA3_TILT 0)" />
     <xacro:property name="tower" value="$(optenv JACKAL_FLEA3_TOWER 1)" />
     <xacro:property name="mount" value="$(optenv JACKAL_FLEA3_MOUNT front)" />

Commit message: set jackal navigate with low scan

File: src/jackal_description/urdf/accessories.urdf.xacro (robot description, xacro)
@@ -109,11 +109,11 @@
   </xacro:if>
   <!-- Secondary 2D Lidar -->
-  <xacro:if value="$(optenv JACKAL_LASER_SECONDARY 0)">
-    <xacro:property name="mount" value="$(optenv JACKAL_LASER_SECONDARY_MOUNT rear)" />
-    <xacro:property name="topic" value="$(optenv JACKAL_LASER_SECONDARY_TOPIC rear/scan)" />
+  <xacro:if value="$(optenv JACKAL_LASER_SECONDARY 1)">
+    <xacro:property name="mount" value="$(optenv JACKAL_LASER_SECONDARY_MOUNT front)" />
+    <xacro:property name="topic" value="$(optenv JACKAL_LASER_SECONDARY_TOPIC front/scan2)" />
     <xacro:property name="tower" value="$(optenv JACKAL_LASER_SECONDARY_TOWER 1)" />
-    <xacro:property name="prefix" value="$(optenv JACKAL_LASER_SECONDARY_PREFIX ${mount})" />
-    <xacro:property name="parent" value="$(optenv JACKAL_LASER_SECONDARY_PARENT ${mount}_mount)" />
-    <xacro:property name="lidar_model" value="$(optenv JACKAL_LASER_SECONDARY_MODEL lms1xx)" />
+    <xacro:property name="prefix" value="$(optenv JACKAL_LASER_SECONDARY_PREFIX ${mount}_low)" />
+    <xacro:property name="parent" value="$(optenv JACKAL_LASER_SECONDARY_PARENT ${mount}_mount_low)" />
+    <xacro:property name="lidar_model" value="$(optenv JACKAL_LASER_SECONDARY_MODEL utm30)" />
     <!-- SICK LMS1xx -->
     <xacro:if value="${lidar_model == 'lms1xx'}">
@@ -159,5 +159,5 @@
     <xacro:if value="${lidar_model == 'utm30'}">
       <xacro:hokuyo_utm30_mount topic="${topic}" prefix="${prefix}" parent_link="${parent}">
-        <origin xyz="$(optenv JACKAL_LASER_SECONDARY_OFFSET 0 0 0)" rpy="$(optenv JACKAL_LASER_SECONDARY_RPY 0 0 3.14159)" />
+        <origin xyz="$(optenv JACKAL_LASER_SECONDARY_OFFSET 0 0 0)" rpy="$(optenv JACKAL_LASER_SECONDARY_RPY 0 0 0)" />
       </xacro:hokuyo_utm30_mount>
     </xacro:if>

File: src/jackal_description/urdf/accessories_one.urdf.xacro (robot description, xacro)
@@ -26,5 +26,5 @@
     optional microstrain IMU's will be added to another frame, by default, "microstrain_link".
   -->
-  <xacro:if value="$(optenv JACKAL_IMU_MICROSTRAIN 1)">
+  <xacro:if value="$(optenv JACKAL_IMU_MICROSTRAIN 0)">
     <xacro:property name="frame"  value="$(optenv JACKAL_IMU_MICROSTRAIN_LINK microstrain_link)"/>
     <xacro:property name="parent" value="$(optenv JACKAL_IMU_MICROSTRAIN_PARENT base_link)"/>
@@ -48,8 +48,8 @@
   <xacro:if value="$(optenv JACKAL_LASER 1)">
     <xacro:property name="mount" value="$(optenv JACKAL_LASER_MOUNT front)" />
-    <xacro:property name="topic" value="$(optenv JACKAL_LASER_TOPIC front/scan1)" />
+    <xacro:property name="topic" value="$(optenv JACKAL_LASER_TOPIC front/scan)" />
     <xacro:property name="tower" value="$(optenv JACKAL_LASER_TOWER 1)" />
-    <xacro:property name="prefix" value="$(optenv JACKAL_LASER_PREFIX ${mount}_high)" />
-    <xacro:property name="parent" value="$(optenv JACKAL_LASER_PARENT ${mount}_mount_high)" />
+    <xacro:property name="prefix" value="$(optenv JACKAL_LASER_PREFIX ${mount})" />
+    <xacro:property name="parent" value="$(optenv JACKAL_LASER_PARENT ${mount}_mount)" />
     <xacro:property name="lidar_model" value="$(optenv JACKAL_LASER_MODEL lms1xx)" />
     <xacro:property name="mount_type" value="$(optenv JACKAL_LASER_MOUNT_TYPE upright)" />
@@ -109,11 +109,11 @@
   </xacro:if>
   <!-- Secondary 2D Lidar -->
-  <xacro:if value="$(optenv JACKAL_LASER_SECONDARY 1)">
-    <xacro:property name="mount" value="$(optenv JACKAL_LASER_SECONDARY_MOUNT front)" />
-    <xacro:property name="topic" value="$(optenv JACKAL_LASER_SECONDARY_TOPIC front/scan2)" />
+  <xacro:if value="$(optenv JACKAL_LASER_SECONDARY 0)">
+    <xacro:property name="mount" value="$(optenv JACKAL_LASER_SECONDARY_MOUNT rear)" />
+    <xacro:property name="topic" value="$(optenv JACKAL_LASER_SECONDARY_TOPIC rear/scan)" />
     <xacro:property name="tower" value="$(optenv JACKAL_LASER_SECONDARY_TOWER 1)" />
-    <xacro:property name="prefix" value="$(optenv JACKAL_LASER_SECONDARY_PREFIX ${mount}_low)" />
-    <xacro:property name="parent" value="$(optenv JACKAL_LASER_SECONDARY_PARENT ${mount}_mount_low)" />
-    <xacro:property name="lidar_model" value="$(optenv JACKAL_LASER_SECONDARY_MODEL utm30)" />
+    <xacro:property name="prefix" value="$(optenv JACKAL_LASER_SECONDARY_PREFIX ${mount})" />
+    <xacro:property name="parent" value="$(optenv JACKAL_LASER_SECONDARY_PARENT ${mount}_mount)" />
+    <xacro:property name="lidar_model" value="$(optenv JACKAL_LASER_SECONDARY_MODEL lms1xx)" />
     <!-- SICK LMS1xx -->
     <xacro:if value="${lidar_model == 'lms1xx'}">
@@ -159,5 +159,5 @@
     <xacro:if value="${lidar_model == 'utm30'}">
       <xacro:hokuyo_utm30_mount topic="${topic}" prefix="${prefix}" parent_link="${parent}">
-        <origin xyz="$(optenv JACKAL_LASER_SECONDARY_OFFSET 0 0 0)" rpy="$(optenv JACKAL_LASER_SECONDARY_RPY 0 0 0)" />
+        <origin xyz="$(optenv JACKAL_LASER_SECONDARY_OFFSET 0 0 0)" rpy="$(optenv JACKAL_LASER_SECONDARY_RPY 0 0 3.14159)" />
       </xacro:hokuyo_utm30_mount>
     </xacro:if>
@@ -262,5 +262,5 @@
   <xacro:if value="$(optenv JACKAL_FLEA3 1)">
     <xacro:property name="name" value="$(optenv JACKAL_FLEA3_NAME front)" />
-    <xacro:property name="tilt" value="$(optenv JACKAL_FLEA3_TILT 0.)" />
+    <xacro:property name="tilt" value="$(optenv JACKAL_FLEA3_TILT 0)" />
     <xacro:property name="tower" value="$(optenv JACKAL_FLEA3_TOWER 1)" />
     <xacro:property name="mount" value="$(optenv JACKAL_FLEA3_MOUNT front)" />

File: src/jackal_description/urdf/jackal.urdf.xacro (robot description, xacro)
@@ -218,4 +218,10 @@
     <origin xyz="${mount_spacing} 0 0" />
   </joint>
+  <link name="front_mount_low"></link>
+  <joint name="front_mount_low_joint" type="fixed">
+    <parent link="mid_mount" />
+    <child link="front_mount_low" />
+    <origin xyz="${mount_spacing} 0 -0.3" />
+  </joint>
   <link name="ultrasonic_sensor_link"></link>
   <joint name="ultrasonic_sensor_joint" type="fixed">

File: src/jackal_description/urdf/jackal_one.urdf.xacro (robot description, xacro)
@@ -218,15 +218,9 @@
     <origin xyz="${mount_spacing} 0 0" />
   </joint>
-  <link name="front_mount_high"></link>
-  <joint name="front_mount_joint_high" type="fixed">
-    <parent link="mid_mount" />
-    <child link="front_mount_high" />
-    <origin xyz="${mount_spacing} 0 0" />
-  </joint>
-  <link name="front_mount_low"></link>
-  <joint name="front_mount_joint_low" type="fixed">
-    <parent link="mid_mount" />
-    <child link="front_mount_low" />
-    <origin xyz="${mount_spacing} 0 -0.3" />
+  <link name="ultrasonic_sensor_link"></link>
+  <joint name="ultrasonic_sensor_joint" type="fixed">
+    <parent link="front_mount"/>
+    <child link="ultrasonic_sensor_link"/>
+    <origin xyz="0.12 0 -0.2" />
   </joint>
   <!-- Bring in simulation data for Gazebo. -->

File: src/velodyne_description/urdf/VLP-16.urdf.xacro (robot description, xacro)
@@ -61,5 +61,5 @@
         <sensor type="gpu_ray" name="${name}-VLP16">
           <pose>0 0 0 0 0 0</pose>
-          <visualize>false</visualize>
+          <visualize>true</visualize>
           <update_rate>${hz}</update_rate>
           <ray>
